File: circuit/_autosave-aircraft.kicad_sch (KiCad schematic)
At the start: 8 parts, among them U1 MCP23017_SP, U2 ESP32, U3 nRF24L01, U4 LCD_Display_20x4, U5 LCD_I2C_Serial, U6 AMS1117-3.3, U7 Joystick_Hall_XY, U8 Joystick_Hall_XY

Commit message: control circuito started, control code started too
Parts:
- added D1, D2, D3, D4: LED, symbol Device:LED
- added SW1, SW10, SW2, SW3, SW4, SW5, SW6, SW7, SW8, SW9: SW_Push_Dual, symbol Switch:SW_Push_Dual
Connections:
- net at U5. (K): now also U4. (K)
- new net: U4. (K), U5. (K) (x15)
Other:
- moved on the sheet: U6
