File: remotecontrol/kicad/control.kicad_sch (KiCad schematic)
At the start: 0 parts

Commit message: remote control schematic done, waiting revision
Parts:
- added C1, C2: 100uF, symbol Device:C_Polarized_US
- added D1, D2, D3, D4, D5: LED, symbol Device:LED
- added R1, R2, R3, R4, R5: 330, symbol Device:R_US
- added RV1: 10K, symbol Device:R_Potentiometer
- added SW1: SW_Push, symbol Switch:SW_Push
- added SW10, SW11, SW2, SW3, SW4, SW5, SW6, SW7, SW8, SW9: SW_Push_Dual, symbol Switch:SW_Push_Dual
- added U1: Battery, symbol airplane_comps:Battery
- added U10, U7: AMS1117-3.3, Package_TO_SOT_SMD:SOT-223-3_TabPin2, symbol Regulator_Linear:AMS1117-3.3
- added U11: Serial_I2C_Module, symbol airplane_comps:Serial_I2C_Module
- added U12: MCP23017_SP, Package_DIP:DIP-28_W7.62mm, symbol Interface_Expansion:MCP23017_SP
- added U13: LCD_20x4, symbol airplane_comps:LCD_20x4
- added U2: ESP32_DevKit, symbol airplane_comps:ESP32_DevKit
- added U3, U4: Joystick_Hall, symbol airplane_comps:Joystick_Hall
- added U5: nRF24L01+, symbol airplane_comps:nRF24L01+
- added U6: ADS1115IDGS, Package_SO:TSSOP-10_3x3mm_P0.5mm, symbol Analog_ADC:ADS1115IDGS
- added U8: Level_Shifter_Bidirectional, symbol airplane_comps:Level_Shifter_Bidirectional
- added U9: L7805, symbol Regulator_Linear:L7805
Connections:
- new net: D1.1 (K), R1.2
- new net: D1.2 (A), U12.27 (GPA6)
- new net: SW1.1, U1.2 (VCC)
- new net: D2.1 (K), R2.2
- new net: SW5.2, U12.22 (GPA1)
- new net: D5.1 (K), R5.2
- new net: U11.4 (SCL), U6.10 (SCL), U8.1 (TXO)
- new net: U3.3 (VX), U6.4 (AIN0)
- new net: U3.4 (VY), U6.5 (AIN1)
- new net: U4.3 (VX), U6.6 (AIN2)
- new net: U4.4 (VY), U6.7 (AIN3)
- new net: C2.1, RV1.1, U11.2 (VCC), U3.1 (VCC), U4.1 (VCC), U6.8 (VDD), U8.4 (HV), U9.3 (OUT)
- new net: U11.3 (SDA), U6.9 (SDA), U8.6 (TXO)
- new net: SW7.2, U12.2 (GPB1)
- new net: U2.11 (GPIO14), U3.5 (PB)
- new net: SW11.2, U12.6 (GPB5)
- new net: SW6.2, U12.1 (GPB0)
- new net: D3.1 (K), R3.2
- new net: D3.2 (A), U12.25 (GPA4)
- new net: U11.5 (VSS), U13.1 (VSS)
- new net: U11.14 (D3), U13.10 (D3)
- new net: U11.15 (D4), U13.11 (D4)
- new net: U11.16 (D5), U13.12 (D5)
- new net: U11.17 (D6), U13.13 (D6)
- new net: U11.18 (D7), U13.14 (D7)
- new net: U11.19 (A), U13.15 (A)
- new net: U11.20 (K), U13.16 (K)
- new net: U11.6 (VDD), U13.2 (VDD)
- new net: U11.7 (V0), U13.3 (V0)
- new net: U11.8 (RS), U13.4 (RS)
- new net: U11.9 (RW), U13.5 (RW)
- new net: U11.10 (E), U13.6 (E)
- new net: U11.11 (D0), U13.7 (D0)
- new net: U11.12 (D1), U13.8 (D1)
- new net: U11.13 (D2), U13.9 (D2)
- new net: SW9.2, U12.4 (GPB3)
- new net: U10.2 (VO), U12.18 (~{RESET}), U12.9 (VDD)
- new net: C1.1, SW1.2, U10.3 (VI), U2.15 (VIN), U7.3 (VI), U9.1 (IN)
- new net: D4.1 (K), R4.2
- new net: D4.2 (A), U12.24 (GPA3)
- new net: SW8.2, U12.3 (GPB2)
- new net: SW3.2, U12.8 (GPB7)
- new net: U2.10 (GPIO27), U4.5 (PB)
- new net: RV1.2, U2.12 (GPIO12)
- new net: U2.16 (GPIO23), U5.6 (MOSI)
- new net: U12.12 (SCK), U2.17 (GPIO22), U8.7 (TXI)
- new net: U12.13 (SDA), U2.20 (GPIO21), U8.12 (TXI)
- new net: U2.21 (GPIO19), U5.7 (MISO)
- new net: U2.22 (GPIO18), U5.5 (SCK)
- new net: U2.26 (GPIO4), U5.3 (CE)
- new net: U2.27 (GPIO2), U5.4 (CSN)
- new net: U2.30 (3.3v), U8.10 (LV)
- new net: SW2.2, U12.7 (GPB6)
- new net: U5.2 (VCC), U7.2 (VO)
- new net: SW4.2, U12.21 (GPA0)
- new net: D5.2 (A), U12.23 (GPA2)
- new net: D2.2 (A), U12.26 (GPA5)
- new net: SW10.2, U12.5 (GPB4)
- new net GND: C1.2, C2.2, R1.1, R2.1, R3.1, R4.1, R5.1, RV1.3, SW10.1, SW11.1, SW2.1, SW3.1, SW4.1, SW5.1, SW6.1, SW7.1, SW8.1, SW9.1, U1.1 (GND), U10.1 (GND), U11.1 (GND), U12.10 (VSS), U12.15 (A0), U12.16 (A1), U12.17 (A2), U2.14 (GND), U2.29 (GND), U3.2 (GND), U4.2 (GND), U5.1 (GND), U6.1 (ADDR), U6.3 (GND), U7.1 (GND), U8.3 (GND), U8.9 (GND), U9.2 (GND)
- no-connect marks 0 -> 45
Other:
- note added: "5 LEDs to general purpose"
- note added: "6 push buttons to navigation over menus 4 push buttons for general purpose"
- note added: "Again, those AMS1117 already have decoupling capacitors because they are a THT module"
- note added: "As the LCD occupies so much pins, we'll use the Serial_I2C module to use I2C instead"
- note added: "Both modules ADS1115 and Serial_I2C are supplied with 5V and their I2C pins maintain that voltage so we need to put that through a level shifter to send to ESP32."
- note added: "I probably gonna use 6 AA batteries totalizing 9V and 2000mAh"
- note added: "If we supply 3.3v to MCP23017 the output will follow. So we maintain the 3.3v restriction to ESP32 over the I2C line. For simplicity we are gonna use the internal pull up resistors"
- note added: "Potentiometer for general purpose (probably engine throttle)"
- note added: "The ESP32 default ADC have 12 bits and ADS1115 have 16 bits of precision These joysticks use 5V by default so we gonna use ADS1115 because of I2C protocol"
- company: (none) -> Breno Soares Alves
- title: (none) -> Remote Control

Commit message: remote control partial pcb done, need to verify joystick and pot dimensions, also need professor check
Parts:
- C1, C2: footprint (none) -> Capacitor_THT:CP_Radial_D5.0mm_P2.00mm
- D1, D2, D3, D4, D5: footprint (none) -> LED_THT:LED_D3.0mm
- R1, R2, R3, R4, R5: footprint (none) -> Resistor_THT:R_Axial_DIN0204_L3.6mm_D1.6mm_P5.08mm_Horizontal
- RV1: footprint (none) -> airplane_foots:Potentiometer_PCB_Connector_3x5.08
- SW1: footprint (none) -> airplane_foots:Toggle_Switch
- SW10, SW11, SW2, SW3, SW4, SW5, SW6, SW7, SW8, SW9: footprint (none) -> Button_Switch_THT:SW_PUSH_6mm_H4.3mm
- U1: footprint (none) -> TerminalBlock:TerminalBlock_bornier-2_P5.08mm
- U10, U7: footprint Package_TO_SOT_SMD:SOT-223-3_TabPin2 -> Connector_PinHeader_2.54mm:PinHeader_1x03_P2.54mm_Vertical
- U11: footprint (none) -> airplane_foots:Serial_I2C_Module
- U13: footprint (none) -> airplane_foots:LCD_Display_20x4
- U2: footprint (none) -> airplane_foots:ESP32_DevKit
- U3, U4: footprint (none) -> airplane_foots:XDCR_COM-09032
- U5: footprint (none) -> airplane_foots:nRF24L01+
- U6: footprint Package_SO:TSSOP-10_3x3mm_P0.5mm -> airplane_foots:ADS1115
- U8: footprint (none) -> airplane_foots:Level_Shifter
- U9: footprint (none) -> Package_TO_SOT_THT:TO-220-3_Horizontal_TabDown
Changed lines of the file:
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@@
 			)
 		)
-		(property "Footprint" ""
+		(property "Footprint" "LED_THT:LED_D3.0mm"
 			(at 20.32 168.91 0)
 			(effects
@@
 			)
 		)
-		(property "Footprint" ""
+		(property "Footprint" "TerminalBlock:TerminalBlock_bornier-2_P5.08mm"
 			(at 34.29 48.26 0)
 			(effects
@@
 			)
 		)
-		(property "Footprint" ""
+		(property "Footprint" "Resistor_THT:R_Axial_DIN0204_L3.6mm_D1.6mm_P5.08mm_Horizontal"
 			(at 30.226 161.544 90)
 			(effects
@@
 			)
 		)
-		(property "Footprint" ""
+		(property "Footprint" "Button_Switch_THT:SW_PUSH_6mm_H4.3mm"
 			(at 151.13 173.99 0)
 			(effects
@@
 			)
 		)
-		(property "Footprint" ""
+		(property "Footprint" "Resistor_THT:R_Axial_DIN0204_L3.6mm_D1.6mm_P5.08mm_Horizontal"
 			(at 56.896 161.544 90)
 			(effects
@@
 			)
 		)
-		(property "Footprint" "Package_SO:TSSOP-10_3x3mm_P0.5mm"
+		(property "Footprint" "airplane_foots:ADS1115"
 			(at 107.95 59.69 0)
 			(effects
@@
 			)
 		)
-		(property "Footprint" ""
+		(property "Footprint" "Button_Switch_THT:SW_PUSH_6mm_H4.3mm"
 			(at 172.72 114.3 0)
 			(effects
@@
 			)
 		)
-		(property "Footprint" ""
+		(property "Footprint" "airplane_foots:XDCR_COM-09032"
 			(at 77.47 46.99 0)
 			(effects
@@
 			)
 		)
-		(property "Footprint" ""
+		(property "Footprint" "Button_Switch_THT:SW_PUSH_6mm_H4.3mm"
 			(at 193.04 130.81 0)
 			(effects
@@
 			)
 		)
-		(property "Footprint" ""
+		(property "Footprint" "Button_Switch_THT:SW_PUSH_6mm_H4.3mm"
 			(at 172.72 97.79 0)
 			(effects
@@
 			)
 		)
-		(property "Footprint" ""
+		(property "Footprint" "Resistor_THT:R_Axial_DIN0204_L3.6mm_D1.6mm_P5.08mm_Horizontal"
 			(at 21.336 161.544 90)
 			(effects
@@
 			)
 		)
-		(property "Footprint" ""
+		(property "Footprint" "LED_THT:LED_D3.0mm"
 			(at 38.1 168.91 0)
 			(effects
@@
 			)
 		)
-		(property "Footprint" ""
+		(property "Footprint" "airplane_foots:LCD_Display_20x4"
 			(at 260.35 45.72 0)
 			(effects
@@
 			)
 		)
-		(property "Footprint" ""
+		(property "Footprint" "Button_Switch_THT:SW_PUSH_6mm_H4.3mm"
 			(at 193.04 97.79 0)
 			(effects
@@
 			)
 		)
-		(property "Footprint" "Package_TO_SOT_SMD:SOT-223-3_TabPin2"
+		(property "Footprint" "Connector_PinHeader_2.54mm:PinHeader_1x03_P2.54mm_Vertical"
 			(at 207.01 76.2 0)
 			(effects
@@
 			)
 		)
-		(property "Footprint" ""
+		(property "Footprint" "LED_THT:LED_D3.0mm"
 			(at 46.99 168.91 0)
 			(effects
@@
 			)
 		)
-		(property "Footprint" ""
+		(property "Footprint" "Button_Switch_THT:SW_PUSH_6mm_H4.3mm"
 			(at 172.72 130.81 0)
 			(effects
@@
 			)
 		)
-		(property "Footprint" ""
+		(property "Footprint" "Button_Switch_THT:SW_PUSH_6mm_H4.3mm"
 			(at 134.62 173.99 0)
 			(effects
@@
 			)
 		)
-		(property "Footprint" ""
+		(property "Footprint" "airplane_foots:ESP32_DevKit"
 			(at 45.72 101.6 0)
 			(effects
@@
 			)
 		)
-		(property "Footprint" ""
+		(property "Footprint" "Button_Switch_THT:SW_PUSH_6mm_H4.3mm"
 			(at 134.62 156.21 0)
 			(effects
@@
 			)
 		)
-		(property "Footprint" "Package_TO_SOT_SMD:SOT-223-3_TabPin2"
+		(property "Footprint" "Connector_PinHeader_2.54mm:PinHeader_1x03_P2.54mm_Vertical"
 			(at 115.57 161.29 0)
 			(effects
@@
 			)
 		)
-		(property "Footprint" ""
+		(property "Footprint" "Resistor_THT:R_Axial_DIN0204_L3.6mm_D1.6mm_P5.08mm_Horizontal"
 			(at 39.116 161.544 90)
 			(effects
@@
 			)
 		)
-		(property "Footprint" ""
+		(property "Footprint" "Package_TO_SOT_THT:TO-220-3_Horizontal_TabDown"
 			(at 160.655 27.94 0)
 			(effects
@@
 			)
 		)
-		(property "Footprint" ""
+		(property "Footprint" "airplane_foots:Serial_I2C_Module"
 			(at 242.57 45.72 0)
 			(effects
@@
 			)
 		)
-		(property "Footprint" ""
+		(property "Footprint" "airplane_foots:XDCR_COM-09032"
 			(at 77.47 62.23 0)
 			(effects
@@
 			)
 		)
-		(property "Footprint" ""
+		(property "Footprint" "airplane_foots:Level_Shifter"
 			(at 157.48 69.85 0)
 			(effects
@@
 			)
 		)
-		(property "Footprint" ""
+		(property "Footprint" "airplane_foots:nRF24L01+"
 			(at 77.47 166.37 0)
 			(effects
@@
 			)
 		)
-		(property "Footprint" ""
+		(property "Footprint" "Capacitor_THT:CP_Radial_D5.0mm_P2.00mm"
 			(at 167.64 27.94 0)
 			(effects
@@
 			)
 		)
-		(property "Footprint" ""
+		(property "Footprint" "airplane_foots:Potentiometer_PCB_Connector_3x5.08"
 			(at 44.45 135.89 0)
 			(effects
@@
 			)
 		)
-		(property "Footprint" ""
+		(property "Footprint" "Button_Switch_THT:SW_PUSH_6mm_H4.3mm"
 			(at 193.04 114.3 0)
 			(effects
@@
 			)
 		)
-		(property "Footprint" ""
+		(property "Footprint" "LED_THT:LED_D3.0mm"
 			(at 55.88 168.91 0)
 			(effects
@@
 			)
 		)
-		(property "Footprint" ""
+		(property "Footprint" "Resistor_THT:R_Axial_DIN0204_L3.6mm_D1.6mm_P5.08mm_Horizontal"
 			(at 48.006 161.544 90)
 			(effects
@@
 			)
 		)
-		(property "Footprint" ""
+		(property "Footprint" "Capacitor_THT:CP_Radial_D5.0mm_P2.00mm"
 			(at 152.4 27.94 0)
 			(effects
@@
 			)
 		)
-		(property "Footprint" ""
+		(property "Footprint" "LED_THT:LED_D3.0mm"
 			(at 29.21 168.91 0)
 			(effects
@@
 			)
 		)
-		(property "Footprint" ""
+		(property "Footprint" "airplane_foots:Toggle_Switch"
 			(at 46.99 45.72 0)
 			(effects
@@
 			)
 		)
-		(property "Footprint" ""
+		(property "Footprint" "Button_Switch_THT:SW_PUSH_6mm_H4.3mm"
 			(at 151.13 156.21 0)
 			(effects

Commit message: remote control done need inspection
Parts:
- added C3, C4: 10uF, Capacitor_THT:CP_Radial_D5.0mm_P2.00mm, symbol Device:C_Polarized_US
- added U14: AMS1117-1.8, Package_TO_SOT_SMD:SOT-223-3_TabPin2, symbol Regulator_Linear:AMS1117-1.8
- U3, U4: footprint airplane_foots:XDCR_COM-09032 -> airplane_foots:Joystick_Hall_Ginfull
Connections:
- net GND: now also C3.2, C4.2, U14.1 (GND)
- net at SW1.1, U1.2 (VCC): now also C1.1, SW1.2, U10.3 (VI), U2.15 (VIN), U7.3 (VI), U9.1 (IN), C4.1, U14.3 (VI)
- net at U6.4 (AIN0): now also U4.4 (VY); no longer U3.3 (VX)
- net at U6.5 (AIN1): now also U4.3 (VX); no longer U3.4 (VY)
- net at U6.6 (AIN2): now also U3.4 (VY); no longer U4.3 (VX)
- net at U6.7 (AIN3): now also U3.3 (VX); no longer U4.4 (VY)
- net at C2.1, RV1.1, U11.2 (VCC)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: no longer U3.1 (VCC), U4.1 (VCC)
- net at U3.5 (PB): now also U2.12 (GPIO12); no longer U2.11 (GPIO14)
- net at RV1.2: now also U2.11 (GPIO14); no longer U2.12 (GPIO12)
- new net: C3.1, U14.2 (VO), U3.1 (VCC), U4.1 (VCC)
