File: remotecontrol/kicad/control.kicad_pcb (KiCad board)
At the start: 2 copper layers, 165 x 123.9 mm, 38 parts, among them SW1 SW_Push, SW10 SW_Push_Dual, SW11 SW_Push_Dual, SW2 SW_Push_Dual, SW3 SW_Push_Dual, SW4 SW_Push_Dual, SW5 SW_Push_Dual, SW6 SW_Push_Dual, SW7 SW_Push_Dual, SW8 SW_Push_Dual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

Commit message: remote control done need inspection
Parts:
- added C3: 10uF, Capacitor_THT:CP_Radial_D5.0mm_P2.00mm, F.Cu at (139.0, 72.9)
- added C4: 10uF, Capacitor_THT:CP_Radial_D5.0mm_P2.00mm, F.Cu at (139.4, 80.5)
- added U14: AMS1117-1.8, Package_TO_SOT_SMD:SOT-223-3_TabPin2, F.Cu at (146.7, 80.5)
- U3, U4: footprint airplane_foots:XDCR_COM-09032 -> airplane_foots:Joystick_Hall_Ginfull
- moved U11 9.18 mm to (112.0, 72.5)
- moved RV1 5.85 mm to (212.5, 99.4)
Connections:
- C1 pad 1: Net-(U10-VI) -> Net-(U1-VCC)
- RV1 pad 2: Net-(U2-GPIO12) -> Net-(U2-GPIO14)
- SW1 pad 2: Net-(U10-VI) -> Net-(U1-VCC)
- U10 pad 3: Net-(U10-VI) -> Net-(U1-VCC)
- U2 pad 15: Net-(U10-VI) -> Net-(U1-VCC)
- U6 pad 4: Net-(U3-VX) -> Net-(U4-VY)
- U6 pad 5: Net-(U3-VY) -> Net-(U4-VX)
- U6 pad 6: Net-(U4-VX) -> Net-(U3-VY)
- U6 pad 7: Net-(U4-VY) -> Net-(U3-VX)
- U7 pad 3: Net-(U10-VI) -> Net-(U1-VCC)
- U9 pad 1: Net-(U10-VI) -> Net-(U1-VCC)
Routing:
- net Net-(U1-VCC): track 8.38 -> 332.6 mm
- net Net-(U10-VI): track 265.6 -> 0.00 mm
- net Net-(U14-VO): track 0.00 -> 215.9 mm
- net Net-(U11-VCC): track 95.3 -> 256.3 mm
- net Net-(U3-VX): track 0.00 -> 155.9 mm
- net Net-(U3-VY): track 0.00 -> 143.5 mm
- net Net-(U2-GPIO27): track 0.00 -> 142.3 mm, vias 0 -> 1
- net Net-(U2-GPIO12): track 0.00 -> 108.6 mm
- net Net-(U4-VY): track 0.00 -> 98.8 mm
- net Net-(U4-VX): track 0.00 -> 94.0 mm
- net Net-(U2-GPIO14): track 0.00 -> 64.7 mm
- net Net-(U11-RS): track 6.50 -> 14.3 mm
- net Net-(U11-RW): track 6.50 -> 13.9 mm
- net Net-(U11-V0): track 6.50 -> 13.9 mm
- net Net-(U11-E): track 6.50 -> 13.6 mm
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