File: kicad/airplane.kicad_sch (KiCad schematic)
At the start: 23 parts, among them M1 Ailerons, M2 Elevator, M3 Rudder, M4 Wheel, U1 ESP32_DevKit, U10 L7805, U11 BMP280, U12 NEO-6M_GPS, U13 SD_Module, U2 nRF24L01+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

Commit message: airplane full pcb done
Parts:
- removed C5, C6: 10uF, Capacitor_THT:CP_Radial_D4.0mm_P1.50mm, symbol Device:C_Polarized
- removed U10: L7805, Package_TO_SOT_THT:TO-220-3_Vertical, symbol Regulator_Linear:L7805
- added R1, R2, R3, R4: 330, Resistor_THT:R_Axial_DIN0204_L3.6mm_D1.6mm_P5.08mm_Horizontal, symbol Device:R_US
- added U10: AMS1117-3.3, Connector_PinHeader_2.54mm:PinHeader_1x03_P2.54mm_Vertical, symbol Regulator_Linear:AMS1117-3.3
Connections:
- net GND: now also U6.3 (GND), U7.3 (GND), R1.2, R2.2, R3.2, R4.2, U10.1 (GND); no longer U6.2 (GND), U7.2 (GND), U8.2 (GNDR), U8.4 (GNDG), U8.6 (GND1), U8.8 (GND2)
- net at C4.1, M3.2 (+), M4.2 (+): now also U7.2 (OUT); no longer U7.3 (OUT)
- net at U11.1 (VCC), U11.5 (CSB), U12.1 (VCC)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: now also U13.2 (3V3), U10.2 (VO); no longer U13.3 (5V)
- net at C2.1, M1.2 (+), M2.2 (+): now also U6.2 (OUT); no longer U6.3 (OUT)
- net at C1.1, C3.1, U5.2 (12v)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: now also U10.3 (VI)
- new net: R2.1, U8.4 (GNDG)
- new net: R4.1, U8.8 (GND2)
- new net: R1.1, U8.2 (GNDR)
- new net: R3.1, U8.6 (GND1)

Commit message: fabrication files created, waiting revision yet
Parts:
- added R5: 1k, Resistor_THT:R_Axial_DIN0204_L3.6mm_D1.6mm_P5.08mm_Horizontal, symbol Device:R_US
- added R6: 620, Resistor_THT:R_Axial_DIN0204_L3.6mm_D1.6mm_P5.08mm_Horizontal, symbol Device:R_US
- added R7: 2k2, Resistor_THT:R_Axial_DIN0204_L3.6mm_D1.6mm_P5.08mm_Horizontal, symbol Device:R_US
Connections:
- net GND: now also R5.2
- net at U1.8 (GPIO25): now also R5.1, R6.2
- net at C1.1, C3.1, U10.3 (VI)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: now also R7.1
- new net: R6.1, R7.2
- no-connect marks 16 -> 15
